File: DIGDuino/DIGDuino.sch (KiCad schematic (older format))
At the start: 34 parts

Commit message: Finished Schematic Design
Schematic Rv1 finished, footprints added
Parts:
- removed P? (x2): CONN_01X12, symbol CONN_01X12
- removed P? (x2): CONN_01X08, symbol CONN_01X08
- added P2, P3: CONN_01X20, symbol CONN_01X20
- added P7: CONN_01X03, symbol CONN_01X03
- C4: renamed from C?; value 1.1n -> 1n
- JP1: renamed from JP?; value Jumper_NC_Small -> USB_Power_En
- gave numbers to parts that had none: 28
Connections:
- net +3V3: now also P2.17 (P17), P2.18 (P18), P3.5 (P5), P3.6 (P6), P3.7 (P7)
- net GND: now also P1.6 (shield), P2.19 (P19), P2.20 (P20), P3.2 (P2), P3.3 (P3), P3.4 (P4), P7.3 (P3)
- net Pin1: now also U2.1 (P6.0/CB0/A0), P2.1 (P1)
- net Pin10: now also U2.15 (TA0.0/P1.1), P2.10 (P10)
- net Pin11: now also U2.16 (TA0.1/P1.2), P2.11 (P11)
- net Pin12: now also U2.17 (TA0.2/P1.3), P2.12 (P12)
- net Pin13: now also U2.18 (TA0.3/P1.4), P2.13 (P13)
- net Pin14: now also U2.19 (TA0.4/P1.5), P2.14 (P14)
- net Pin15: now also U2.20 (TA1CLK/CBOUT/P1.6), P2.15 (P15)
- net Pin16: now also U2.21 (TA1.0/P1.7), P2.16 (P16)
- net Pin17: now also U2.22 (TA1.1/P2.0), P3.20 (P20)
- net Pin18: now also U2.23 (PJ.0/TDO), P3.19 (P19)
- net Pin19: now also U2.24 (PJ.1/TDI/TCLK), P3.18 (P18)
- net Pin2: now also U2.2 (P6.1/CB1/A1), P2.2 (P2)
- net Pin20: now also U2.25 (PJ.2/TMS), P3.17 (P17)
- net Pin21: now also U2.26 (PJ.3/TCK), P3.16 (P16)
- net Pin22: now also U2.29 (PM_UCB1STE/PM_UCA1CLK/P4.0), P3.15 (P15)
- net Pin23: now also U2.30 (PM_UCB1SIMO/PM_UCB1SDA/P4.1), P3.14 (P14)
- net Pin24: now also U2.31 (PM_UCB1SOMI/PM_UCB1SCL/P4.2), P3.13 (P13)
- net Pin25: now also U2.32 (PM_UCB1CLK/PM_UCA1STE/P4.3), P3.12 (P12)
- net Pin26: now also U2.33 (PM_UCA1TXD/PM_UCA1SIMO/P4.4), P3.11 (P11)
- net Pin27: now also U2.34 (PM_UCA1RXD/PM_UCA1SOMI/P4.5), P3.10 (P10)
- net Pin28: now also U2.35 (P4.6), P3.9 (P9)
- net Pin29: now also U2.36 (P4.7), P3.8 (P8)
- net Pin3: now also U2.3 (P6.2/CB2/A2), P2.3 (P3)
- net Pin4: now also U2.4 (P6.3/CB3/A3), P2.4 (P4)
- net Pin5: now also U2.5 (P5.0/A8/VeREF+), P2.5 (P5)
- net Pin6: now also U2.6 (P5.1/A9/VeREF-), P2.6 (P6)
- net Pin7: now also U2.8 (P5.4/XIN), P2.7 (P7)
- net Pin8: now also U2.9 (P5.5/XOUT), P2.8 (P8)
- net Pin9: now also U2.14 (TA0CLK/ACLK/P1.0), P2.9 (P9)
- net RST: now also P7.1 (P1)
- net TCK: now also P7.2 (P2)
- net Vin: now also P3.1 (P1)
